Commit message: [WIP] Adds rotation constraints

File: robots/j2s6s200.urdf (robot description, URDF)
Before this commit: robot j2s6s200, 14 links, 13 joints
Joints:
- joint j2s6s200_joint_end_effector: origin xyz=0 0 -0.1600 rpy=3.14159265359 0 1.57079632679 -> xyz=0 0 -0.1600 rpy=3.14159265359 1.57079632679 0
